File: usb_dongle_hw/usb_dongle_hw.kicad_sch (KiCad schematic)
At the start: 35 parts, among them U1 RP2040, U1 W25Q64JV, U2 AP2112K-3.3, Y1 12Mhz

Commit message: feat: DRC pass, routing complete
Parts:
- added TP1: TestPoint, TestPoint:TestPoint_Pad_D1.0mm, symbol CM4IO:TestPoint
Connections:
- net GND: now also TP1.1
- net usb-d-: now reaches R7.2, U1.46 (USB_D-)
- net usb-d+: now reaches R7.2, U1.47 (USB_D+)
Other:
- moved on the sheet: R7
Changed lines of the file:
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@@
     (stroke (width 0) (type default))
   )
-  (wire (pts (xy 40.005 59.055) (xy 41.529 59.055))
-    (stroke (width 0) (type default))
-  )
-  (wire (pts (xy 46.609 56.515) (xy 48.26 56.515))
+  (wire (pts (xy 32.639 58.674) (xy 34.163 58.674))
     (stroke (width 0) (type default))
   )
@@
     (stroke (width 0) (type default))
   )
-  (wire (pts (xy 40.005 56.515) (xy 41.529 56.515))
+  (wire (pts (xy 32.639 56.134) (xy 34.163 56.134))
     (stroke (width 0) (type default))
   )
@@
   )
   (wire (pts (xy 144.78 78.105) (xy 144.78 83.185))
-    (stroke (width 0) (type default))
-  )
-  (wire (pts (xy 46.609 59.055) (xy 48.26 59.055))
     (stroke (width 0) (type default))
   )
@@
   (text "Conn." (at 173.101 68.072 0)
     (effects (font (size 6 6)) (justify left bottom))
+  )
+  (label "usb-d-" (at 39.243 58.674 0) (fields_autoplaced)
+    (effects (font (size 1.27 1.27)) (justify left bottom))
+  )
+  (label "usb-d+" (at 39.243 56.134 0) (fields_autoplaced)
+    (effects (font (size 1.27 1.27)) (justify left bottom))
+  )
+  (label "usb-d+" (at 48.26 56.515 0) (fields_autoplaced)
+    (effects (font (size 1.27 1.27)) (justify left bottom))
+  )
+  (label "usb-d-" (at 48.26 59.055 0) (fields_autoplaced)
+    (effects (font (size 1.27 1.27)) (justify left bottom))
   )
   (global_label "QSPI_SD0" (shape input) (at 48.26 71.755 180) (fields_autoplaced)
@@
     )
   )
-  (global_label "USB_d+" (shape input) (at 40.005 56.515 180) (fields_autoplaced)
+  (global_label "USB_d+" (shape input) (at 32.639 56.134 180) (fields_autoplaced)
     (effects (font (size 1.27 1.27)) (justify right))
-    (property "Intersheetrefs" "${INTERSHEET_REFS}" (at 29.5208 56.515 0)
+    (property "Intersheetrefs" "${INTERSHEET_REFS}" (at 22.1548 56.134 0)
       (effects (font (size 1.27 1.27)) (justify right) hide)
     )
@@
     )
   )
-  (global_label "USB_d-" (shape input) (at 40.005 59.055 180) (fields_autoplaced)
+  (global_label "USB_d-" (shape input) (at 32.639 58.674 180) (fields_autoplaced)
     (effects (font (size 1.27 1.27)) (justify right))
-    (property "Intersheetrefs" "${INTERSHEET_REFS}" (at 29.5208 59.055 0)
+    (property "Intersheetrefs" "${INTERSHEET_REFS}" (at 22.1548 58.674 0)
       (effects (font (size 1.27 1.27)) (justify right) hide)
     )
@@
     )
   )
-  (symbol (lib_id "Device:R_Small") (at 44.069 59.055 90) (unit 1)
+  (symbol (lib_id "Device:R_Small") (at 36.703 58.674 90) (unit 1)
     (in_bom yes) (on_board yes) (dnp no)
-    (property "Reference" "R7" (at 48.006 61.849 90)
-      (effects (font (size 1.27 1.27)) (justify left))
-    )
-    (property "Value" "27" (at 44.831 61.722 90)
-      (effects (font (size 1.27 1.27)) (justify left))
-    )
-    (property "Footprint" "Resistor_SMD:R_0603_1608Metric" (at 44.069 59.055 0)
-      (effects (font (size 1.27 1.27)) hide)
-    )
-    (property "Datasheet" "~" (at 44.069 59.055 0)
+    (property "Reference" "R7" (at 40.64 61.468 90)
+      (effects (font (size 1.27 1.27)) (justify left))
+    )
+    (property "Value" "27" (at 37.465 61.341 90)
+      (effects (font (size 1.27 1.27)) (justify left))
+    )
+    (property "Footprint" "Resistor_SMD:R_0603_1608Metric" (at 36.703 58.674 0)
+      (effects (font (size 1.27 1.27)) hide)
+    )
+    (property "Datasheet" "~" (at 36.703 58.674 0)
       (effects (font (size 1.27 1.27)) hide)
     )
@@
     )
   )
+  (symbol (lib_id "CM4IO:TestPoint") (at 215.646 72.136 0) (unit 1)
+    (in_bom yes) (on_board yes) (dnp no) (fields_autoplaced)
+    (property "Reference" "TP1" (at 218.186 67.564 0)
+      (effects (font (size 1.27 1.27)) (justify left))
+    )
+    (property "Value" "TestPoint" (at 218.186 70.104 0)
+      (effects (font (size 1.27 1.27)) (justify left))
+    )
+    (property "Footprint" "TestPoint:TestPoint_Pad_D1.0mm" (at 220.726 72.136 0)
+      (effects (font (size 1.27 1.27)) hide)
+    )
+    (property "Datasheet" "~" (at 220.726 72.136 0)
+      (effects (font (size 1.27 1.27)) hide)
+    )
+    (pin "1")
+    (instances
+      (project "airolit_mav_eth_serial_bridge"
+        (path "/b6aa0f6e-488c-4abb-84ec-08259f32154f"
+          (reference "TP1") (unit 1)
+        )
+      )
+      (project "usb_dongle_hw"
+        (path "/f1e8cca5-6520-4615-9bd0-ed3c9e2daac7"
+          (reference "TP8") (unit 1)
+        )
+      )
+    )
+  )
   (symbol (lib_id "power:GND") (at 113.03 112.395 90) (unit 1)
     (in_bom yes) (on_board yes) (dnp no) (fields_autoplaced)
@@
     )
   )
-  (symbol (lib_id "Device:R_Small") (at 44.069 56.515 90) (unit 1)
+  (symbol (lib_id "Device:R_Small") (at 36.703 56.134 90) (unit 1)
     (in_bom yes) (on_board yes) (dnp no)
-    (property "Reference" "R7" (at 48.26 52.959 90)
-      (effects (font (size 1.27 1.27)) (justify left))
-    )
-    (property "Value" "27" (at 45.466 54.356 90)
-      (effects (font (size 1.27 1.27)) (justify left))
-    )
-    (property "Footprint" "Resistor_SMD:R_0603_1608Metric" (at 44.069 56.515 0)
-      (effects (font (size 1.27 1.27)) hide)
-    )
-    (property "Datasheet" "~" (at 44.069 56.515 0)
+    (property "Reference" "R7" (at 40.894 52.578 90)
+      (effects (font (size 1.27 1.27)) (justify left))
+    )
+    (property "Value" "27" (at 38.1 53.975 90)
+      (effects (font (size 1.27 1.27)) (justify left))
+    )
+    (property "Footprint" "Resistor_SMD:R_0603_1608Metric" (at 36.703 56.134 0)
+      (effects (font (size 1.27 1.27)) hide)
+    )
+    (property "Datasheet" "~" (at 36.703 56.134 0)
       (effects (font (size 1.27 1.27)) hide)
     )
@@
         )
       )
+    )
+  )
+  (symbol (lib_id "power:GND") (at 215.646 72.136 0) (unit 1)
+    (in_bom yes) (on_board yes) (dnp no) (fields_autoplaced)
+    (property "Reference" "#PWR021" (at 215.646 78.486 0)
+      (effects (font (size 1.27 1.27)) hide)
+    )
+    (property "Value" "GND" (at 215.646 77.216 0)
+      (effects (font (size 1.27 1.27)))
+    )
+    (property "Footprint" "" (at 215.646 72.136 0)
+      (effects (font (size 1.27 1.27)) hide)
+    )
+    (property "Datasheet" "" (at 215.646 72.136 0)
+      (effects (font (size 1.27 1.27)) hide)
+    )
+    (pin "1")
+    (instances
+      (project "rp2040_magslide_controller"
+        (path "/3d4d216d-def1-4055-8a0c-d95415001574"
+          (reference "#PWR021") (unit 1)
+        )
+      )
+      (project "airolit_mav_eth_serial_bridge"
+        (path "/b6aa0f6e-488c-4abb-84ec-08259f32154f"
+          (reference "#PWR01") (unit 1)
+        )
+      )
+      (project "usb_dongle_hw"
+        (path "/f1e8cca5-6520-4615-9bd0-ed3c9e2daac7"
+          (reference "#PWR031") (unit 1)
+        )
+      )
