File: usb_dongle_hw/usb_dongle_hw.kicad_pcb (KiCad board)
At the start: 2 copper layers, 12 x 28 mm, 35 parts, among them U1 RP2040, U2 W25Q64JV, U3 AP2112K-3.3, Y1 12Mhz

Commit message: wip
Parts:
- moved C11 1.05 mm to (75.1, 105.9)
- moved R3 1.05 mm to (73.0, 105.9)
- moved U2 1.05 mm to (74.2, 108.1)
- moved R4 1.05 mm to (77.9, 106.3)
Changed lines of the file:
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@@
   )
   (footprint "Resistor_SMD:R_0402_1005Metric" (layer "F.Cu")
-    (at 73.025 104.874)
+    (at 73.025 105.922)
     (descr "Resistor SMD 0402 (1005 Metric), square (rectangular) end terminal, IPC_7351 nominal, (Body size source: IPC-SM-782 page 72, https://www.pcb-3d.com/wordpress/wp-content/uploads/ipc-sm-782a_amendment_1_and_2.pdf), generated with kicad-footprint-generator")
     (tags "resistor")
@@
   )
   (footprint "Capacitor_SMD:C_0402_1005Metric" (layer "F.Cu")
-    (at 75.057 104.874)
+    (at 75.057 105.922)
     (descr "Capacitor SMD 0402 (1005 Metric), square (rectangular) end terminal, IPC_7351 nominal, (Body size source: IPC-SM-782 page 76, https://www.pcb-3d.com/wordpress/wp-content/uploads/ipc-sm-782a_amendment_1_and_2.pdf), generated with kicad-footprint-generator")
     (tags "capacitor")
@@
   )
   (footprint "Resistor_SMD:R_0402_1005Metric" (layer "F.Cu")
-    (at 77.851 105.253 90)
+    (at 77.851 106.299 90)
     (descr "Resistor SMD 0402 (1005 Metric), square (rectangular) end terminal, IPC_7351 nominal, (Body size source: IPC-SM-782 page 72, https://www.pcb-3d.com/wordpress/wp-content/uploads/ipc-sm-782a_amendment_1_and_2.pdf), generated with kicad-footprint-generator")
     (tags "resistor")
@@
   )
   (footprint "Library:SON50P300X200X60-9N" (layer "F.Cu")
-    (at 74.165 107.033)
+    (at 74.165 108.081)
     (descr "<b>USON 2x3x0.6-mm</b><br>")
     (property "Sheetfile" "usb_dongle_hw.kicad_sch")

Commit message: feat: DRC pass, routing complete
Parts:
- added TP8: TestPoint, TestPoint:TestPoint_Pad_D1.0mm, B.Cu at (77.9, 113.4)
- TP1, TP2, TP3, TP4, TP5, TP6, TP7: moved to B.Cu
- moved TP3 112.5 mm to (80.0, 115.4), turned to 180 degrees
- moved TP4 111.2 mm to (77.9, 115.4), turned to 180 degrees
- moved TP1 109.0 mm to (80.0, 113.3), turned to 180 degrees
- moved TP7 106.0 mm to (77.9, 104.0), turned to 180 degrees
- moved TP5 104.7 mm to (77.9, 101.9), turned to 180 degrees
- moved TP6 100.9 mm to (80.1, 101.9), turned to 180 degrees
- moved TP2 98.8 mm to (80.1, 104.0), turned to 180 degrees
Connections:
- net Net-(U1-USB_DM) renamed /usb-d-
- net Net-(U1-USB_DP) renamed /usb-d+
Routing:
- net +3V3: track 0.00 -> 88.0 mm, vias 0 -> 8
- net GND: track 0.00 -> 56.2 mm, vias 0 -> 12
- net +5V: track 0.00 -> 40.3 mm, vias 0 -> 3
- net +1V1: track 0.00 -> 22.1 mm, vias 0 -> 2
- net /usb-d+: track 0.00 -> 10.8 mm, vias 0 -> 2
- net /usb-d-: track 0.00 -> 10.7 mm, vias 0 -> 2
- net Net-(U1-XIN): track 0.00 -> 8.21 mm
- net QSPI_CS: track 0.00 -> 8.18 mm
- net QSPI_SD1: track 0.00 -> 7.41 mm, vias 0 -> 2
- net Net-(U1-GPIO25): track 0.00 -> 7.10 mm, vias 0 -> 2
- net Net-(U1-XOUT): track 0.00 -> 6.27 mm
- net USB_d-: track 0.00 -> 5.97 mm, vias 0 -> 1
- net QSPI_SD3: track 0.00 -> 5.88 mm, vias 0 -> 2
- net QSPI_SD2: track 0.00 -> 4.89 mm
- net USB_d+: track 0.00 -> 4.39 mm, vias 0 -> 1
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- added copper zone on B.Cu, net GND
- added copper zone on F.Cu, net GND

Commit message: fix: Silk
Other:
- board text added: "3v3"
- board text added: "5V"
- board text added: "Act"
- board text added: "Gnd"
- board text added: "Ripxospeech Dongle Rev. 1"
- board text added: "d+"
- board text added: "d-"
- board text added: "gnd"
- board text added: "swc"
- board text added: "swd"
Changed lines of the file:
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@@
   (gr_line (start 73.4136 100.4824) (end 81.4136 100.4824)
     (stroke (width 0.1) (type default)) (layer "Edge.Cuts"))
+  (gr_text "3v3" (at 82.042 112.141) (layer "B.SilkS")
+    (effects (font (size 0.75 0.75) (thickness 0.15)) (justify left bottom mirror))
+  )
+  (gr_text "5V" (at 76.708 103.886) (layer "B.SilkS")
+    (effects (font (size 0.75 0.75) (thickness 0.15)) (justify left bottom mirror))
+  )
+  (gr_text "d+" (at 76.9112 101.6) (layer "B.SilkS")
+    (effects (font (size 0.75 0.75) (thickness 0.15)) (justify left bottom mirror))
+  )
+  (gr_text "d-" (at 82.6008 101.6) (layer "B.SilkS")
+    (effects (font (size 0.75 0.75) (thickness 0.15)) (justify left bottom mirror))
+  )
+  (gr_text "Ripxospeech Dongle Rev. 1" (at 72.5932 111.0996 90) (layer "B.SilkS")
+    (effects (font (size 0.75 0.75) (thickness 0.15)) (justify left bottom mirror))
+  )
+  (gr_text "Gnd" (at 77.343 112.522) (layer "B.SilkS")
+    (effects (font (size 0.75 0.75) (thickness 0.15)) (justify left bottom mirror))
+  )
+  (gr_text "swd" (at 82.55 117.221) (layer "B.SilkS")
+    (effects (font (size 0.75 0.75) (thickness 0.15)) (justify left bottom mirror))
+  )
+  (gr_text "gnd" (at 81.534 105.664) (layer "B.SilkS")
+    (effects (font (size 0.75 0.75) (thickness 0.15)) (justify left bottom mirror))
+  )
+  (gr_text "swc" (at 77.851 117.221) (layer "B.SilkS")
+    (effects (font (size 0.75 0.75) (thickness 0.15)) (justify left bottom mirror))
+  )
+  (gr_text "Act" (at 81.4324 125.1204 -90) (layer "F.SilkS")
+    (effects (font (size 0.75 0.75) (thickness 0.15)) (justify left bottom))
+  )
   (segment (start 80.22 103.108) (end 80.22 102.733) (width 0.18) (layer "F.Cu") (net 1))
   (segment (start 76.594 117.873) (end 76.594 117.353282) (width 0.18) (layer "F.Cu") (net 1))

Commit message: fix: Silk
Other:
- board text added: "rip^rip speech"
- board text removed: "Act"
Changed lines of the file:
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@@
     (effects (font (size 0.75 0.75) (thickness 0.15)) (justify left bottom mirror))
   )
-  (gr_text "Act" (at 81.4324 125.1204 -90) (layer "F.SilkS")
-    (effects (font (size 0.75 0.75) (thickness 0.15)) (justify left bottom))
+  (gr_text "rip^rip\nspeech" (at 80.4164 126.4412 270) (layer "F.SilkS")
+    (effects (font (size 0.75 0.75) (thickness 0.15)) (justify bottom))
   )
   (segment (start 80.22 103.108) (end 80.22 102.733) (width 0.18) (layer "F.Cu") (net 1))
